File: TLE8888-1QK.kicad_sch (KiCad schematic)
At the start: 8 parts, among them Q1 IPD30N06S2L-23

Commit message: First commit
Parts:
- removed C10: 100nF, Capacitor_SMD:C_0603_1608Metric, symbol Device:C
- removed C11: 4.7nF, Capacitor_SMD:C_0603_1608Metric, symbol Device:C
- removed C9: 10uF, Capacitor_SMD:C_0603_1608Metric, symbol Device:C
- removed Q1: IPD30N06S2L-23, Package_TO_SOT_SMD:TO-252-2, symbol Transistor_FET:BUZ11
- added 10u1: L_Small, symbol Device:L_Small
- added 2.2u1: INDUCTOR, symbol pspice:INDUCTOR
- added C1: 4.7u, Capacitor_SMD:C_0603_1608Metric, symbol Device:C
- added C3: 1u, Capacitor_SMD:C_0603_1608Metric, symbol Device:C
- added C4: 10n, Capacitor_SMD:C_0603_1608Metric, symbol Device:C
- added C5: 100n, symbol Device:C_Small
- added C6: 270p, Capacitor_SMD:C_0603_1608Metric, symbol Device:C
- added C7: 10u, Capacitor_SMD:C_0603_1608Metric, symbol Device:C
- added D1: D_Schottky, symbol Device:D_Schottky
- added R1: R, symbol Device:R
- added R2: 10k, Resistor_SMD:R_0402_1005Metric, symbol Device:R
- added R3: 12k, Resistor_SMD:R_0402_1005Metric, symbol Device:R
- added R4: 68k, Resistor_SMD:R_0402_1005Metric, symbol Device:R
- added U2: LMR14020, Simon:SOIC8-DFN, symbol Simon:LMR14020
- C8: value 10uF -> 10u; LCSC C19702 -> (none); Manufacturer TDK -> (none); Part # C1608X5R1E106M080AC -> (none); VEND DIGI -> (none); VEND# 445-9015-1-ND -> (none)
Connections:
- net 12V_SAFE: now also 2.2u1.1, R1.1; no longer C2.1
- net GND: now also C1.2, C3.2, C4.2, C7.2, D1.2 (A), R2.2, R3.2, U2.7 (GND), U2.9 (GND)
- net V6V renamed 5V
- net 5V: now also 10u1.2, C6.1, C7.1, R4.1
- new net: 2.2u1.2, C2.1, C3.1, U2.2 (VIN), U2.3 (EN)
- new net: C5.1, U2.1 (BOOT)
- new net: 10u1.1, C5.2, D1.1 (K), U2.8 (SW)
- new net: C1.1, R1.2
- new net: C6.2, R3.1, R4.2, U2.5 (FB)
- new net: R2.1, U2.4 (RT)
- new net: C4.1, U2.6 (SS)
Other:
- moved on the sheet: C2

Commit message: did stuff
Parts:
- 10u1: footprint (none) -> Inductor_SMD:L_1210_3225Metric
- 2.2u1: footprint (none) -> Simon:MWSA0503
- C5: footprint (none) -> Capacitor_SMD:C_0603_1608Metric
- D1: footprint (none) -> Diode_SMD:D_SMA
- R1: value R -> 1; footprint (none) -> Resistor_SMD:R_0402_1005Metric
Changed lines of the file:
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@@
       (effects (font (size 1.27 1.27)) (justify left))
     )
-    (property "Footprint" "" (id 2) (at 327.66 283.21 0)
+    (property "Footprint" "Capacitor_SMD:C_0603_1608Metric" (id 2) (at 327.66 283.21 0)
       (effects (font (size 1.27 1.27)) hide)
     )
@@
       (effects (font (size 1.27 1.27)) (justify left))
     )
-    (property "Value" "R" (id 1) (at 260.35 289.5599 0)
-      (effects (font (size 1.27 1.27)) (justify left))
-    )
-    (property "Footprint" "" (id 2) (at 256.032 288.29 90)
+    (property "Value" "1" (id 1) (at 260.35 289.5599 0)
+      (effects (font (size 1.27 1.27)) (justify left))
+    )
+    (property "Footprint" "Resistor_SMD:R_0402_1005Metric" (id 2) (at 256.032 288.29 90)
       (effects (font (size 1.27 1.27)) hide)
     )
@@
     (property "Reference" "10u1" (id 0) (at 345.44 280.67 90))
     (property "Value" "L_Small" (id 1) (at 345.44 283.21 90))
-    (property "Footprint" "" (id 2) (at 345.44 285.75 0)
+    (property "Footprint" "Inductor_SMD:L_1210_3225Metric" (id 2) (at 345.44 285.75 0)
       (effects (font (size 1.27 1.27)) hide)
     )
@@
     (property "Reference" "2.2u1" (id 0) (at 265.43 273.05 0))
     (property "Value" "INDUCTOR" (id 1) (at 265.43 275.59 0))
-    (property "Footprint" "" (id 2) (at 265.43 279.4 0)
+    (property "Footprint" "Simon:MWSA0503" (id 2) (at 265.43 279.4 0)
       (effects (font (size 1.27 1.27)) hide)
     )
@@
       (effects (font (size 1.27 1.27)) (justify right))
     )
-    (property "Footprint" "" (id 2) (at 335.28 275.59 0)
-      (effects (font (size 1.27 1.27)) hide)
-    )
+    (property "Footprint" "Diode_SMD:D_SMA" (id 2) (at 335.28 275.59 0)
+      (effects (font (size 1.27 1.27)) hide)
+    )
