File: adc.kicad_sch (KiCad schematic)
At the start: 87 parts, among them U35 MCP6004, U36 MCP6004, U46 MCP6004, U8 MCP6004

Commit message: Fixed CAN and 5v pads
Other:
- title: microRusEFI-2L -> MRE IO Expander
Changed lines of the file:
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@@
   (paper "B")
   (title_block
-    (title "microRusEFI-2L")
-    (date "2020-05-24")
-    (rev "R0.5.2")
+    (title "MRE IO Expander")
+    (date "2021-02-")
+    (rev "R0.1")
     (company "rusEFI.com")
-    (comment 1 "Donald Becker")
+    (comment 1 "Simon Orchard")
     (comment 2 "AI6OD")
   )
