File: micro_rusEFI.kicad_sch (KiCad schematic)
At the start: 27 parts, among them J4 Conn_02x05_Counter_Clockwise, U3 molex_48pin_MRE

Commit message: First commit
Parts:
- removed J4: Conn_02x05_Counter_Clockwise, Connector_PinHeader_2.54mm:PinHeader_2x05_P2.54mm_Vertical_SMD, symbol Connector_Generic:Conn_02x05_Odd_Even
- removed R21, R33, R80, R81: 0R, Resistor_SMD:R_0603_1608Metric, symbol Device:R
Other:
- note removed: "Communication Header"
- moved on the sheet: TP12, TP3

Commit message: did stuff
Parts:
- U3: footprint rusefi_lib:Molex_48_MRE -> rusefi_lib:Molex_48_BCM
Changed lines of the file:
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@@
       (effects (font (size 1.524 1.524)))
     )
-    (property "Footprint" "rusefi_lib:Molex_48_MRE" (id 2) (at 196.85 53.975 0)
+    (property "Footprint" "rusefi_lib:Molex_48_BCM" (id 2) (at 196.85 53.975 0)
       (effects (font (size 1.524 1.524)) hide)
     )
@@
       (effects (font (size 1.524 1.524)) hide)
     )
-    (property "Footprint" "rusefi_lib:Molex_48_MRE" (id 2) (at 310.515 33.655 0)
+    (property "Footprint" "rusefi_lib:Molex_48_BCM" (id 2) (at 310.515 33.655 0)
       (effects (font (size 1.524 1.524)) hide)
     )
@@
       (effects (font (size 1.524 1.524)) hide)
     )
-    (property "Footprint" "rusefi_lib:Molex_48_MRE" (id 2) (at 272.415 90.805 0)
+    (property "Footprint" "rusefi_lib:Molex_48_BCM" (id 2) (at 272.415 90.805 0)
       (effects (font (size 1.524 1.524)) hide)
     )
@@
       (effects (font (size 1.524 1.524)) hide)
     )
-    (property "Footprint" "rusefi_lib:Molex_48_MRE" (id 2) (at 178.435 206.375 0)
+    (property "Footprint" "rusefi_lib:Molex_48_BCM" (id 2) (at 178.435 206.375 0)
       (effects (font (size 1.524 1.524)) hide)
     )
@@
       (effects (font (size 1.524 1.524)) hide)
     )
-    (property "Footprint" "rusefi_lib:Molex_48_MRE" (id 2) (at 178.435 203.835 0)
+    (property "Footprint" "rusefi_lib:Molex_48_BCM" (id 2) (at 178.435 203.835 0)
       (effects (font (size 1.524 1.524)) hide)
     )
@@
       (effects (font (size 1.524 1.524)) hide)
     )
-    (property "Footprint" "rusefi_lib:Molex_48_MRE" (id 2) (at 177.8 212.09 0)
+    (property "Footprint" "rusefi_lib:Molex_48_BCM" (id 2) (at 177.8 212.09 0)
       (effects (font (size 1.524 1.524)) hide)
     )
@@
       (effects (font (size 1.524 1.524)) hide)
     )
-    (property "Footprint" "rusefi_lib:Molex_48_MRE" (id 2) (at 195.58 226.695 0)
+    (property "Footprint" "rusefi_lib:Molex_48_BCM" (id 2) (at 195.58 226.695 0)
       (effects (font (size 1.524 1.524)) hide)
     )
@@
       (effects (font (size 1.524 1.524)) hide)
     )
-    (property "Footprint" "rusefi_lib:Molex_48_MRE" (id 2) (at 195.58 234.315 0)
+    (property "Footprint" "rusefi_lib:Molex_48_BCM" (id 2) (at 195.58 234.315 0)
       (effects (font (size 1.524 1.524)) hide)
     )
@@
       (effects (font (size 1.524 1.524)) hide)
     )
-    (property "Footprint" "rusefi_lib:Molex_48_MRE" (id 2) (at 195.58 236.855 0)
+    (property "Footprint" "rusefi_lib:Molex_48_BCM" (id 2) (at 195.58 236.855 0)
       (effects (font (size 1.524 1.524)) hide)
     )
@@
       (effects (font (size 1.524 1.524)) hide)
     )
-    (property "Footprint" "rusefi_lib:Molex_48_MRE" (id 2) (at 195.58 239.395 0)
+    (property "Footprint" "rusefi_lib:Molex_48_BCM" (id 2) (at 195.58 239.395 0)
       (effects (font (size 1.524 1.524)) hide)
     )
@@
       (effects (font (size 1.524 1.524)) hide)
     )
-    (property "Footprint" "rusefi_lib:Molex_48_MRE" (id 2) (at 195.58 231.775 0)
+    (property "Footprint" "rusefi_lib:Molex_48_BCM" (id 2) (at 195.58 231.775 0)
       (effects (font (size 1.524 1.524)) hide)
     )
@@
       (effects (font (size 1.524 1.524)) hide)
     )
-    (property "Footprint" "rusefi_lib:Molex_48_MRE" (id 2) (at 261.62 117.475 0)
+    (property "Footprint" "rusefi_lib:Molex_48_BCM" (id 2) (at 261.62 117.475 0)
       (effects (font (size 1.524 1.524)) hide)
     )
@@
     )
     (path "/00000000-0000-0000-0000-00005c5d7fa6/af0b75b4-a64d-4a5e-8354-9a260f8c98b2"
-      (reference "2.2u1") (unit 1) (value "INDUCTOR") (footprint "")
+      (reference "2.2u1") (unit 1) (value "INDUCTOR") (footprint "Simon:MWSA0503")
     )
     (path "/00000000-0000-0000-0000-00005c5d7fa6/4a59a32d-2b47-4348-8807-b2b43b7d1193"
-      (reference "10u1") (unit 1) (value "L_Small") (footprint "")
+      (reference "10u1") (unit 1) (value "L_Small") (footprint "Inductor_SMD:L_1210_3225Metric")
     )
     (path "/00000000-0000-0000-0000-00005c5d7fa6/f0330e9d-5112-4dc0-b07f-f827e8dc268c"
@@
     )
     (path "/00000000-0000-0000-0000-00005c5d7fa6/057fa376-9d40-441f-8772-43aaae16caf2"
-      (reference "C5") (unit 1) (value "100n") (footprint "")
+      (reference "C5") (unit 1) (value "100n") (footprint "Capacitor_SMD:C_0603_1608Metric")
     )
     (path "/00000000-0000-0000-0000-00005c5d7fa6/6031f4d5-cb06-4042-b7dd-a4c33ea22759"
@@
     )
     (path "/00000000-0000-0000-0000-00005c5d7fa6/c266c5e9-26ce-4324-845a-6fae6489a0be"
-      (reference "D1") (unit 1) (value "D_Schottky") (footprint "")
+      (reference "D1") (unit 1) (value "D_Schottky") (footprint "Diode_SMD:D_SMA")
     )
     (path "/00000000-0000-0000-0000-00005e9b40e4"
@@
     )
     (path "/00000000-0000-0000-0000-00005c5d7fa6/20fcf059-ceaa-40e8-a2b1-5e422a7a34b9"
-      (reference "R1") (unit 1) (value "R") (footprint "")
+      (reference "R1") (unit 1) (value "1") (footprint "Resistor_SMD:R_0402_1005Metric")
     )
     (path "/00000000-0000-0000-0000-00005c5d7fa6/96571ea4-422b-4986-8d5a-19c0547da6ca"
@@
     )
     (path "/00000000-0000-0000-0000-00005dd8bb43"
-      (reference "U3") (unit 1) (value "molex_48pin_MRE") (footprint "rusefi_lib:Molex_48_MRE")
+      (reference "U3") (unit 1) (value "molex_48pin_MRE") (footprint "rusefi_lib:Molex_48_BCM")
     )
     (path "/00000000-0000-0000-0000-00005d0250fb/00000000-0000-0000-0000-00005e8ee3bc"
-      (reference "U3") (unit 3) (value "molex_48pin_MRE") (footprint "rusefi_lib:Molex_48_MRE")
+      (reference "U3") (unit 3) (value "molex_48pin_MRE") (footprint "rusefi_lib:Molex_48_BCM")
     )
     (path "/00000000-0000-0000-0000-00005e7587f2"
-      (reference "U3") (unit 4) (value "molex_48pin_MRE") (footprint "rusefi_lib:Molex_48_MRE")
+      (reference "U3") (unit 4) (value "molex_48pin_MRE") (footprint "rusefi_lib:Molex_48_BCM")
     )
     (path "/00000000-0000-0000-0000-00005e75e517"
-      (reference "U3") (unit 6) (value "molex_48pin_MRE") (footprint "rusefi_lib:Molex_48_MRE")
+      (reference "U3") (unit 6) (value "molex_48pin_MRE") (footprint "rusefi_lib:Molex_48_BCM")
     )
     (path "/00000000-0000-0000-0000-00005d0250fb/00000000-0000-0000-0000-00005ebaf142"
-      (reference "U3") (unit 7) (value "molex_48pin_MRE") (footprint "rusefi_lib:Molex_48_MRE")
+      (reference "U3") (unit 7) (value "molex_48pin_MRE") (footprint "rusefi_lib:Molex_48_BCM")
     )
     (path "/00000000-0000-0000-0000-00005fdea88f"
-      (reference "U3") (unit 8) (value "molex_48pin_MRE") (footprint "rusefi_lib:Molex_48_MRE")
+      (reference "U3") (unit 8) (value "molex_48pin_MRE") (footprint "rusefi_lib:Molex_48_BCM")
     )
     (path "/00000000-0000-0000-0000-00005fe1bbb9"
-      (reference "U3") (unit 9) (value "molex_48pin_MRE") (footprint "rusefi_lib:Molex_48_MRE")
+      (reference "U3") (unit 9) (value "molex_48pin_MRE") (footprint "rusefi_lib:Molex_48_BCM")
     )
     (path "/00000000-0000-0000-0000-00005fe33973"
-      (reference "U3") (unit 10) (value "molex_48pin_MRE") (footprint "rusefi_lib:Molex_48_MRE")
+      (reference "U3") (unit 10) (value "molex_48pin_MRE") (footprint "rusefi_lib:Molex_48_BCM")
     )
     (path "/00000000-0000-0000-0000-00005fe3397d"
-      (reference "U3") (unit 11) (value "molex_48pin_MRE") (footprint "rusefi_lib:Molex_48_MRE")
+      (reference "U3") (unit 11) (value "molex_48pin_MRE") (footprint "rusefi_lib:Molex_48_BCM")
     )
     (path "/00000000-0000-0000-0000-00005fe4fa20"
-      (reference "U3") (unit 12) (value "molex_48pin_MRE") (footprint "rusefi_lib:Molex_48_MRE")
+      (reference "U3") (unit 12) (value "molex_48pin_MRE") (footprint "rusefi_lib:Molex_48_BCM")
     )
     (path "/00000000-0000-0000-0000-00005fe4fa2a"
-      (reference "U3") (unit 13) (value "molex_48pin_MRE") (footprint "rusefi_lib:Molex_48_MRE")
+      (reference "U3") (unit 13) (value "molex_48pin_MRE") (footprint "rusefi_lib:Molex_48_BCM")
     )
     (path "/00000000-0000-0000-0000-00005fe4fa34"
-      (reference "U3") (unit 14) (value "molex_48pin_MRE") (footprint "rusefi_lib:Molex_48_MRE")
+      (reference "U3") (unit 14) (value "molex_48pin_MRE") (footprint "rusefi_lib:Molex_48_BCM")
     )
     (path "/00000000-0000-0000-0000-00005f86e169"
-      (reference "U3") (unit 15) (value "molex_48pin_MRE") (footprint "rusefi_lib:Molex_48_MRE")
+      (reference "U3") (unit 15) (value "molex_48pin_MRE") (footprint "rusefi_lib:Molex_48_BCM")
     )
     (path "/00000000-0000-0000-0000-00005f86bb48"
-      (reference "U3") (unit 16) (value "molex_48pin_MRE") (footprint "rusefi_lib:Molex_48_MRE")
+      (reference "U3") (unit 16) (value "molex_48pin_MRE") (footprint "rusefi_lib:Molex_48_BCM")
     )
     (path "/00000000-0000-0000-0000-00005d0250fb/00000000-0000-0000-0000-00005d8f198d"

Commit message: 5v stage improved
Connections:
- no-connect marks 16 -> 14
Changed lines of the file:
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@@
   (no_connect (at 257.81 29.845))
   (no_connect (at 233.68 28.575))
-  (no_connect (at 273.05 137.795))
   (no_connect (at 219.71 33.655))
-  (no_connect (at 273.05 140.335))
   (no_connect (at 219.71 31.115))
   (no_connect (at 219.71 28.575))
@@
     (stroke (width 0) (type default) (color 0 0 0 0))
   )
+  (wire (pts (xy 212.09 152.4) (xy 212.09 172.085))
+    (stroke (width 0) (type default) (color 0 0 0 0))
+  )
   (wire (pts (xy 338.455 36.195) (xy 340.36 36.195))
     (stroke (width 0) (type default) (color 0 0 0 0))
@@
     (stroke (width 0) (type default) (color 0 0 0 0))
   )
-  (wire (pts (xy 201.93 172.085) (xy 203.835 172.085))
+  (wire (pts (xy 201.93 172.085) (xy 212.09 172.085))
     (stroke (width 0) (type default) (color 0 0 0 0))
   )
@@
   )
   (wire (pts (xy 200.66 41.91) (xy 200.66 40.005))
+    (stroke (width 0) (type default) (color 0 0 0 0))
+  )
+  (wire (pts (xy 228.6 152.4) (xy 212.09 152.4))
     (stroke (width 0) (type default) (color 0 0 0 0))
   )
@@
     (effects (font (size 1.524 1.524) (thickness 0.3048) bold) (justify right bottom))
   )
+  (hierarchical_label "5V" (shape output) (at 228.6 152.4 0)
+    (effects (font (size 1.27 1.27)) (justify left))
+  )
   (symbol (lib_id "Connector:TestPoint") (at 367.665 50.165 270) (unit 1)

Commit message: Started CAN
Other:
- added sheet CAN Transceiver (CAN.kicad_sch)
Changed lines of the file:
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@@
+    )
+  )
+  (sheet (at 97.79 152.4) (size 45.72 25.4) (fields_autoplaced)
+    (stroke (width 0.1524) (type solid) (color 0 0 0 0))
+    (fill (color 0 0 0 0.0000))
+    (property "Sheet name" "CAN Transceiver" (id 0) (at 97.79 151.6884 0)
+      (effects (font (size 1.27 1.27)) (justify left bottom))
+    )
+    (property "Sheet file" "CAN.kicad_sch" (id 1) (at 97.79 178.3846 0)
+      (effects (font (size 1.27 1.27)) (justify left top))
     )
   )
@@
     (path "/" (page "1"))
     (path "/00000000-0000-0000-0000-00005ce2282d" (page "2"))
+    (path "/969a92ae-25d5-4d7d-9e86-53a15c209495" (page "5"))
     (path "/00000000-0000-0000-0000-00005d0250fb" (page "7"))
     (path "/00000000-0000-0000-0000-00005c5d7fa6" (page "8"))
@@
       (reference "#PWR0214") (unit 1) (value "GND") (footprint "")
     )
+    (path "/969a92ae-25d5-4d7d-9e86-53a15c209495/8e6bb250-d07b-4af9-9ac2-79f79142e15f"
+      (reference "#PWR?") (unit 1) (value "GND") (footprint "")
+    )
     (path "/00000000-0000-0000-0000-00005c5d7fa6/af0b75b4-a64d-4a5e-8354-9a260f8c98b2"
       (reference "2.2u1") (unit 1) (value "INDUCTOR") (footprint "Simon:MWSA0503")
@@
       (reference "D42") (unit 1) (value "BAV70") (footprint "Package_TO_SOT_SMD:SOT-23")
     )
+    (path "/969a92ae-25d5-4d7d-9e86-53a15c209495/07a8f2a9-82a1-4a6f-ba50-dea7b0328dd3"
+      (reference "D?") (unit 1) (value "PESD1CAN-UX") (footprint "digikey-footprints:SOT-323")
+    )
     (path "/00000000-0000-0000-0000-00005d0250fb/00000000-0000-0000-0000-00005c470c85"
       (reference "FB1") (unit 1) (value "FILTER") (footprint "Resistor_SMD:R_0603_1608Metric_Pad1.05x0.95mm_HandSolder")
@@
       (reference "R141") (unit 1) (value "10K") (footprint "Resistor_SMD:R_0603_1608Metric")
     )
+    (path "/969a92ae-25d5-4d7d-9e86-53a15c209495/62f34f0e-e660-4f65-a8b8-bf9ce863bcd8"
+      (reference "R?") (unit 1) (value "R") (footprint "")
+    )
     (path "/00000000-0000-0000-0000-00005cf9a0a2"
       (reference "RN1") (unit 1) (value "1k") (footprint "Resistor_SMD:R_Array_Convex_4x0603")
@@
       (reference "U46") (unit 5) (value "MCP6004") (footprint "Package_SO:TSSOP-14_4.4x5mm_P0.65mm")
     )
+    (path "/969a92ae-25d5-4d7d-9e86-53a15c209495/7627e349-e05f-47f1-bd34-5e7e2a92ccbc"
+      (reference "U?") (unit 1) (value "TJA1051T-3") (footprint "Package_SO:SOIC-8_3.9x4.9mm_P1.27mm")
+    )
     (path "/00000000-0000-0000-0000-00005d0250fb/00000000-0000-0000-0000-000052d13afb"
