File: Six_Axis.kicad_sch (KiCad schematic)
At the start: 3 parts

Commit message: Work on 6 axis
Parts:
- gave numbers to parts that had none: 3
Connections:
- net SDO: now reaches U10.1 (SDO/SA0)
- net CS: now reaches U10.12 (CS)
- net SCK: now reaches U10.13 (SCL)
- net SDI: now reaches U10.14 (SDA)
Changed lines of the file:
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@@
     (stroke (width 0) (type default) (color 0 0 0 0))
   )
-  (wire (pts (xy 100.33 96.52) (xy 121.92 96.52))
+  (wire (pts (xy 105.41 96.52) (xy 121.92 96.52))
     (stroke (width 0) (type default) (color 0 0 0 0))
   )
@@
     (stroke (width 0) (type default) (color 0 0 0 0))
   )
-  (wire (pts (xy 100.33 81.28) (xy 121.92 81.28))
+  (wire (pts (xy 105.41 81.28) (xy 121.92 81.28))
     (stroke (width 0) (type default) (color 0 0 0 0))
   )
   (wire (pts (xy 139.7 63.5) (xy 139.7 69.85))
     (stroke (width 0) (type default) (color 0 0 0 0))
+  )
+  (global_label "SCK" (shape input) (at 105.41 93.98 180) (fields_autoplaced)
+    (effects (font (size 1.27 1.27)) (justify right))
+    (property "Intersheet References" "${INTERSHEET_REFS}" (id 0) (at 99.3363 93.9006 0)
+      (effects (font (size 1.27 1.27)) (justify right) hide)
+    )
+  )
+  (global_label "SDO" (shape input) (at 105.41 81.28 180) (fields_autoplaced)
+    (effects (font (size 1.27 1.27)) (justify right))
+    (property "Intersheet References" "${INTERSHEET_REFS}" (id 0) (at 99.2758 81.2006 0)
+      (effects (font (size 1.27 1.27)) (justify right) hide)
+    )
+  )
+  (global_label "CS" (shape input) (at 105.41 96.52 180) (fields_autoplaced)
+    (effects (font (size 1.27 1.27)) (justify right))
+    (property "Intersheet References" "${INTERSHEET_REFS}" (id 0) (at 100.6063 96.4406 0)
+      (effects (font (size 1.27 1.27)) (justify right) hide)
+    )
+  )
+  (global_label "SDI" (shape input) (at 105.41 91.44 180) (fields_autoplaced)
+    (effects (font (size 1.27 1.27)) (justify right))
+    (property "Intersheet References" "${INTERSHEET_REFS}" (id 0) (at 100.0015 91.3606 0)
+      (effects (font (size 1.27 1.27)) (justify right) hide)
+    )
   )
   (global_label "VDD" (shape input) (at 139.7 63.5 90) (fields_autoplaced)
@@
   (symbol (lib_id "power:GND") (at 137.16 104.14 0) (unit 1)
     (in_bom yes) (on_board yes) (fields_autoplaced)
-    (property "Reference" "#PWR?" (id 0) (at 137.16 110.49 0)
+    (property "Reference" "#PWR0164" (id 0) (at 137.16 110.49 0)
       (effects (font (size 1.27 1.27)) hide)
     )
@@
   (symbol (lib_id "Sensor_Motion:LSM6DS3") (at 137.16 88.9 0) (unit 1)
     (in_bom yes) (on_board yes) (fields_autoplaced)
-    (property "Reference" "U?" (id 0) (at 154.94 74.7012 0))
+    (property "Reference" "U10" (id 0) (at 154.94 74.7012 0))
     (property "Value" "LSM6DS3" (id 1) (at 154.94 77.2412 0))
     (property "Footprint" "Package_LGA:LGA-14_3x2.5mm_P0.5mm_LayoutBorder3x4y" (id 2) (at 127 106.68 0)
@@
   (symbol (lib_id "Device:C_Small") (at 128.27 67.31 0) (unit 1)
     (in_bom yes) (on_board yes) (fields_autoplaced)
-    (property "Reference" "C?" (id 0) (at 130.81 66.0462 0)
+    (property "Reference" "C13" (id 0) (at 130.81 66.0462 0)
       (effects (font (size 1.27 1.27)) (justify left))
     )
@@
   (symbol (lib_id "Device:C_Small") (at 143.51 69.85 90) (unit 1)
     (in_bom yes) (on_board yes) (fields_autoplaced)
-    (property "Reference" "C?" (id 0) (at 143.5163 63.5 90))
+    (property "Reference" "C14" (id 0) (at 143.5163 63.5 90))
     (property "Value" "100nF" (id 1) (at 143.5163 66.04 90))
     (property "Footprint" "Capacitor_SMD:C_0402_1005Metric" (id 2) (at 143.51 69.85 0)
@@
   (symbol (lib_id "power:GND") (at 146.05 69.85 90) (unit 1)
     (in_bom yes) (on_board yes) (fields_autoplaced)
-    (property "Reference" "#PWR?" (id 0) (at 152.4 69.85 0)
+    (property "Reference" "#PWR0162" (id 0) (at 152.4 69.85 0)
       (effects (font (size 1.27 1.27)) hide)
     )
@@
   (symbol (lib_id "power:GND") (at 128.27 69.85 0) (unit 1)
     (in_bom yes) (on_board yes) (fields_autoplaced)
-    (property "Reference" "#PWR?" (id 0) (at 128.27 76.2 0)
+    (property "Reference" "#PWR0160" (id 0) (at 128.27 76.2 0)
       (effects (font (size 1.27 1.27)) hide)
     )
@@
   (symbol (lib_id "power:GND") (at 139.7 104.14 0) (unit 1)
     (in_bom yes) (on_board yes) (fields_autoplaced)
-    (property "Reference" "#PWR?" (id 0) (at 139.7 110.49 0)
+    (property "Reference" "#PWR0167" (id 0) (at 139.7 110.49 0)
       (effects (font (size 1.27 1.27)) hide)
     )
@@
   (symbol (lib_id "power:GND") (at 96.52 83.82 0) (unit 1)
     (in_bom yes) (on_board yes)
-    (property "Reference" "#PWR?" (id 0) (at 96.52 90.17 0)
+    (property "Reference" "#PWR0161" (id 0) (at 96.52 90.17 0)
       (effects (font (size 1.27 1.27)) hide)
     )
